File: kicad_files/33RPI23_rp3_case.kicad_pcb (KiCad board)
At the start: 2 copper layers, 56 x 85 mm, 112 parts, among them CN1 locked, J1 VGA, J10 AudioJack4, J11 USB_B_Micro, J12 Mini-DIN-6, J13 Mini-DIN-6, J14 Conn_01x07, J15 Conn_01x01_Female, J16 USB, J17 Conn_01x02_Female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

Commit message: labels
Parts:
- added J20: Conn_01x02, Connector_PinHeader_2.54mm:PinHeader_1x02_P2.54mm_Vertical, F.Cu at (35.7, 74.0)
- added R44: 10k, Resistor_SMD:R_0805_2012Metric_Pad1.20x1.40mm_HandSolder, B.Cu at (44.0, 88.6)
- moved R13 4.78 mm to (50.0, 92.5), turned to -90 degrees
- moved R19 3.59 mm to (73.4, 65.1)
- moved R25 1.44 mm to (73.4, 56.7)
- moved J3 1.37 mm to (38.2, 76.6)
Routing:
- net Net-(J20-Pad2): track 0.00 -> 18.1 mm, vias 0 -> 1
- net GND: track 603.2 -> 613.1 mm
- net /R_U: track 18.0 -> 8.53 mm
- net Net-(C12-Pad1): track 45.8 -> 53.7 mm
- net /D+: track 39.9 -> 32.4 mm
- net /RIGHT_OUT: track 6.14 -> 9.99 mm
- net /R_OUT: track 28.8 -> 32.4 mm
- net /+5V: track 588.2 -> 591.4 mm
- net Net-(C9-Pad1): track 15.8 -> 14.1 mm
- net Net-(C6-Pad1): track 15.2 -> 13.6 mm
- net /D-: track 35.7 -> 37.2 mm
- net /BEEP_OUT: track 26.7 -> 28.1 mm
- net /GP_21: track 14.9 -> 13.6 mm
- net /LEFT_OUT: track 5.61 -> 6.84 mm
- net /VGA_RH: track 20.5 -> 19.6 mm
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Other:
- board text added: "0"
- board text added: "1"
- board text added: "10"
- board text added: "11"
- board text added: "12"
- board text added: "13"
- board text added: "2"
- board text added: "3"
- board text added: "4"
- board text added: "5"
- board text added: "6"
- board text added: "7"
- board text added: "8"
- board text added: "9"
- board text added: "C20"
- board text added: "I"
- board text added: "IN"
- board text added: "OUT"

Commit message: l2
Parts:
- added G***: LOGO, LOGO, F.Cu at (54.6, 109.1)
- C14: value 10u -> 100u
- R1, R2, R3, R4, R5, R6, R7, R8: moved to B.Cu
- moved R37 1.30 mm to (73.3, 49.1)
- moved R27 0.64 mm to (73.7, 60.2)
- moved G*** 0.13 mm to (54.6, 109.0)
- renumbered C1 to C1*
Routing:
- net /GP_4: track 26.4 -> 39.6 mm
- net Net-(C12-Pad1): track 53.7 -> 65.0 mm
- net /VGA_BL: track 19.9 -> 28.0 mm
- net /GP_2: track 25.5 -> 28.5 mm
- net /VGA_RL: track 33.4 -> 31.6 mm
- net /VGA_GL: track 23.4 -> 22.0 mm
- net /RST: track 29.4 -> 30.8 mm
- net /GP_5: track 39.1 -> 39.9 mm
- net /+3V3: track 104.5 -> 105.2 mm
- net GND: track 613.1 -> 612.5 mm
- net /+3V3A: track 102.5 -> 101.9 mm
- net /GP_23_3v3EN: track 14.3 -> 14.8 mm
Other:
- board text added: "+3V"
- board text added: "14"
- board text added: "15"
- board text added: "16"
- board text added: "17"
- board text added: "18"
- board text added: "19"
- board text added: "20"
- board text added: "21"
- board text added: "22"
- board text added: "23*"
- board text added: "26"
- board text added: "27"
- board text added: "28"
- board text added: "29*"
- board text added: "A.IN"
- board text added: "A.OUT"
- board text added: "B"
- board text added: "G"
- board text added: "HS"
- board text added: "PS2_C"
- board text added: "PS2_D"
- board text added: "RST"
- board text added: "VS"
- board text removed: "3V3"
- board text removed: "OUT"

Commit message: +jumpers
USB PS/2 jumpers
Parts:
- added JP10: J, Jumper:SolderJumper-2_P1.3mm_Open_RoundedPad1.0x1.5mm, B.Cu at (59.2, 96.5)
- added JP11: J, Jumper:SolderJumper-2_P1.3mm_Open_RoundedPad1.0x1.5mm, B.Cu at (61.5, 96.5)
- added JP12: J, Jumper:SolderJumper-2_P1.3mm_Open_RoundedPad1.0x1.5mm, B.Cu at (73.5, 105.0)
- added JP13: J, Jumper:SolderJumper-2_P1.3mm_Open_RoundedPad1.0x1.5mm, B.Cu at (71.5, 105.0)
Connections:
- J8 pad 6: /DM3 -> Net-(J8-Pad6)
- J8 pad 7: /DP3 -> Net-(J8-Pad7)
Routing:
- net Net-(J8-Pad7): track 0.00 -> 19.2 mm
- net /DP3: track 25.6 -> 8.24 mm
- net Net-(J8-Pad6): track 0.00 -> 16.9 mm, vias 0 -> 1
- net /DM3: track 25.0 -> 8.95 mm, vias 1 -> 0
- net /PS/2 DATA: track 71.5 -> 74.6 mm
- net /PS/2 CLK: track 74.5 -> 77.1 mm, vias 3 -> 4
- net /+5V: track 591.4 -> 589.3 mm
- net /R_OUT: track 32.4 -> 31.5 mm
- net /DM2: track 34.8 -> 34.3 mm
- net GND: track 612.5 -> 613.0 mm
Other:
- board text added: "+3VA"

Commit message: .
Parts:
- added J21: Conn_01x01_Female, Connector_Pin:Pin_D0.7mm_L6.5mm_W1.8mm_FlatFork, B.Cu at (32.9, 32.4)
- added R45: 300, Resistor_SMD:R_0805_2012Metric_Pad1.20x1.40mm_HandSolder, B.Cu at (34.8, 30.6)
Routing:
- net GND: track 613.0 -> 630.7 mm
- net Net-(J21-Pad1): track 0.00 -> 2.15 mm
- net /VGA_VS: track 57.2 -> 58.1 mm
- net /VGA_HS: track 52.3 -> 53.2 mm
- net Net-(D6-Pad2): track 4.95 -> 5.70 mm

Commit message: usb comb
Parts:
- moved G*** 4.45 mm to (60.3, 85.5)
- turned C12 to 90 degrees
Routing:
- net Net-(C12-Pad1): track 65.0 -> 58.8 mm, vias 4 -> 2
- net Net-(C12-Pad2): track 10.7 -> 7.91 mm
