File: kicad_files/33RPI23_rp3_case.kicad_sch (KiCad schematic)
At the start: 110 parts, among them CN1 HDMI, J1 VGA, J10 AudioJack4, J11 USB_B_Micro, J12 Mini-DIN-6, J13 Mini-DIN-6, J14 Conn_01x07, J15 Conn_01x01_Female, J16 USB, J17 Conn_01x02_Female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

Commit message: +jumpers
USB PS/2 jumpers
Parts:
- added JP10, JP11, JP12, JP13: J, Jumper:SolderJumper-2_P1.3mm_Open_RoundedPad1.0x1.5mm, symbol Jumper:SolderJumper_2_Open
Connections:
- net DM3: now also JP11.2 (B); no longer J8.6 (D2-)
- net DP3: now also JP10.2 (B); no longer J8.7 (D2+)
- net PS/2 CLK: now also JP12.2 (B)
- net PS/2 DATA: now also JP13.2 (B)
- new net: J8.6 (D2-), JP11.1 (A), JP13.1 (A)
- new net: J8.7 (D2+), JP10.1 (A), JP12.1 (A)
Changed lines of the file:
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@@
   (junction (at 224.79 241.3) (diameter 0) (color 0 0 0 0)
   )
+  (junction (at 193.04 144.78) (diameter 0) (color 0 0 0 0)
+  )
   (junction (at 121.92 142.24) (diameter 0) (color 0 0 0 0)
   )
@@
   (junction (at 269.24 173.99) (diameter 0) (color 0 0 0 0)
   )
+  (junction (at 195.58 137.16) (diameter 0) (color 0 0 0 0)
+  )
   (junction (at 35.56 234.95) (diameter 0) (color 0 0 0 0)
   )
@@
   (no_connect (at 229.87 59.69))
   (no_connect (at 229.87 41.91))
-  (wire (pts (xy 229.87 123.19) (xy 233.68 123.19))
+  (wire (pts (xy 195.58 127) (xy 195.58 137.16))
     (stroke (width 0) (type default) (color 0 0 0 0))
   )
-  (wire (pts (xy 190.5 129.54) (xy 200.66 129.54))
+  (wire (pts (xy 229.87 123.19) (xy 233.68 123.19))
     (stroke (width 0) (type default) (color 0 0 0 0))
   )
@@
     (stroke (width 0) (type default) (color 0 0 0 0))
   )
+  (wire (pts (xy 199.39 140.97) (xy 195.58 140.97))
+    (stroke (width 0) (type default) (color 0 0 0 0))
+  )
   (wire (pts (xy 229.87 91.44) (xy 229.87 93.98))
     (stroke (width 0) (type default) (color 0 0 0 0))
@@
     (stroke (width 0) (type default) (color 0 0 0 0))
   )
+  (wire (pts (xy 207.01 148.59) (xy 218.44 148.59))
+    (stroke (width 0) (type default) (color 0 0 0 0))
+  )
   (wire (pts (xy 219.71 241.3) (xy 224.79 241.3))
     (stroke (width 0) (type default) (color 0 0 0 0))
   )
+  (wire (pts (xy 195.58 140.97) (xy 195.58 137.16))
+    (stroke (width 0) (type default) (color 0 0 0 0))
+  )
   (wire (pts (xy 219.71 257.81) (xy 226.06 257.81))
     (stroke (width 0) (type default) (color 0 0 0 0))
@@
     (stroke (width 0) (type default) (color 0 0 0 0))
   )
+  (wire (pts (xy 193.04 148.59) (xy 199.39 148.59))
+    (stroke (width 0) (type default) (color 0 0 0 0))
+  )
   (wire (pts (xy 166.37 181.61) (xy 158.75 181.61))
     (stroke (width 0) (type default) (color 0 0 0 0))
@@
     (stroke (width 0) (type default) (color 0 0 0 0))
   )
-  (wire (pts (xy 190.5 127) (xy 200.66 127))
-    (stroke (width 0) (type default) (color 0 0 0 0))
-  )
   (wire (pts (xy 229.87 105.41) (xy 229.87 101.6))
     (stroke (width 0) (type default) (color 0 0 0 0))
@@
     (stroke (width 0) (type default) (color 0 0 0 0))
   )
+  (wire (pts (xy 195.58 137.16) (xy 199.39 137.16))
+    (stroke (width 0) (type default) (color 0 0 0 0))
+  )
   (wire (pts (xy 162.56 242.57) (xy 162.56 245.11))
     (stroke (width 0) (type default) (color 0 0 0 0))
@@
     (stroke (width 0) (type default) (color 0 0 0 0))
   )
+  (wire (pts (xy 207.01 137.16) (xy 218.44 137.16))
+    (stroke (width 0) (type default) (color 0 0 0 0))
+  )
   (wire (pts (xy 144.78 99.06) (xy 144.78 95.25))
     (stroke (width 0) (type default) (color 0 0 0 0))
@@
     (stroke (width 0) (type default) (color 0 0 0 0))
   )
+  (wire (pts (xy 207.01 140.97) (xy 218.44 140.97))
+    (stroke (width 0) (type default) (color 0 0 0 0))
+  )
   (wire (pts (xy 151.13 63.5) (xy 163.83 63.5))
     (stroke (width 0) (type default) (color 0 0 0 0))
@@
     (stroke (width 0) (type default) (color 0 0 0 0))
   )
+  (wire (pts (xy 190.5 129.54) (xy 193.04 129.54))
+    (stroke (width 0) (type default) (color 0 0 0 0))
+  )
   (wire (pts (xy 208.28 91.44) (xy 218.44 91.44))
     (stroke (width 0) (type default) (color 0 0 0 0))
@@
     (stroke (width 0) (type default) (color 0 0 0 0))
   )
+  (wire (pts (xy 207.01 144.78) (xy 218.44 144.78))
+    (stroke (width 0) (type default) (color 0 0 0 0))
+  )
   (wire (pts (xy 30.48 134.62) (xy 46.99 134.62))
     (stroke (width 0) (type default) (color 0 0 0 0))
@@
     (stroke (width 0) (type default) (color 0 0 0 0))
   )
+  (wire (pts (xy 193.04 129.54) (xy 193.04 144.78))
+    (stroke (width 0) (type default) (color 0 0 0 0))
+  )
   (wire (pts (xy 205.74 48.26) (xy 205.74 44.45))
     (stroke (width 0) (type default) (color 0 0 0 0))
@@
     (stroke (width 0) (type default) (color 0 0 0 0))
   )
+  (wire (pts (xy 190.5 127) (xy 195.58 127))
+    (stroke (width 0) (type default) (color 0 0 0 0))
+  )
   (wire (pts (xy 59.69 165.1) (xy 76.2 165.1))
     (stroke (width 0) (type default) (color 0 0 0 0))
@@
     (stroke (width 0) (type default) (color 0 0 0 0))
   )
+  (wire (pts (xy 193.04 144.78) (xy 199.39 144.78))
+    (stroke (width 0) (type default) (color 0 0 0 0))
+  )
   (wire (pts (xy 219.71 154.94) (xy 236.22 154.94))
     (stroke (width 0) (type default) (color 0 0 0 0))
@@
     (stroke (width 0) (type default) (color 0 0 0 0))
   )
+  (wire (pts (xy 193.04 144.78) (xy 193.04 148.59))
+    (stroke (width 0) (type default) (color 0 0 0 0))
+  )
   (wire (pts (xy 142.24 95.25) (xy 139.7 95.25))
     (stroke (width 0) (type default) (color 0 0 0 0))
@@
     (effects (font (size 1.27 1.27)) (justify left bottom))
   )
+  (label "PS{slash}2 CLK" (at 208.28 140.97 0)
+    (effects (font (size 1.27 1.27)) (justify left bottom))
+  )
   (label "GND" (at 33.02 19.05 0)
     (effects (font (size 1.27 1.27)) (justify left bottom))
@@
     (effects (font (size 1.27 1.27)) (justify left bottom))
   )
+  (label "PS{slash}2 DATA" (at 208.28 148.59 0)
+    (effects (font (size 1.27 1.27)) (justify left bottom))
+  )
   (label "GP_11" (at 113.03 55.88 0)
     (effects (font (size 1.27 1.27)) (justify left bottom))
@@
     (effects (font (size 1.27 1.27)) (justify left bottom))
   )
-  (label "DP3" (at 193.04 127 0)
+  (label "DP3" (at 208.28 137.16 0)
     (effects (font (size 1.27 1.27)) (justify left bottom))
   )
@@
     (effects (font (size 1.27 1.27)) (justify left bottom))
   )
-  (label "DM3" (at 193.04 129.54 0)
+  (label "DM3" (at 208.28 144.78 0)
     (effects (font (size 1.27 1.27)) (justify left bottom))
   )
@@
     (pin "1")
   )
+  (symbol (lib_id "Jumper:SolderJumper_2_Open") (at 203.2 148.59 0) (unit 1)
+    (in_bom yes) (on_board yes)
+    (property "Reference" "JP13" (id 0) (at 199.39 147.32 0))
+    (property "Value" "J" (id 1) (at 207.01 147.32 0)
+      (effects (font (size 1.27 1.27)) hide)
+    )
+    (property "Footprint" "Jumper:SolderJumper-2_P1.3mm_Open_RoundedPad1.0x1.5mm" (id 2) (at 203.2 148.59 0)
+      (effects (font (size 1.27 1.27)) hide)
+    )
+    (property "Datasheet" "~" (id 3) (at 203.2 148.59 0)
+      (effects (font (size 1.27 1.27)) hide)
+    )
+    (pin "1")
+    (pin "2")
+  )
   (symbol (lib_id "Device:C") (at 203.2 114.3 270) (unit 1)
     (in_bom yes) (on_board yes)
@@
     (pin "1")
   )
+  (symbol (lib_id "Jumper:SolderJumper_2_Open") (at 203.2 144.78 0) (unit 1)
+    (in_bom yes) (on_board yes)
+    (property "Reference" "JP11" (id 0) (at 199.39 143.51 0))
+    (property "Value" "J" (id 1) (at 207.01 143.51 0)
+      (effects (font (size 1.27 1.27)) hide)
+    )
+    (property "Footprint" "Jumper:SolderJumper-2_P1.3mm_Open_RoundedPad1.0x1.5mm" (id 2) (at 203.2 144.78 0)
+      (effects (font (size 1.27 1.27)) hide)
+    )
+    (property "Datasheet" "~" (id 3) (at 203.2 144.78 0)
+      (effects (font (size 1.27 1.27)) hide)
+    )
+    (pin "1")
+    (pin "2")
+  )
   (symbol (lib_id "Connector:AudioJack4") (at 214.63 160.02 0) (mirror x) (unit 1)
     (in_bom yes) (on_board yes) (fields_autoplaced)
@@
     (pin "2")
   )
+  (symbol (lib_id "Jumper:SolderJumper_2_Open") (at 203.2 137.16 0) (unit 1)
+    (in_bom yes) (on_board yes)
+    (property "Reference" "JP10" (id 0) (at 199.39 135.89 0))
+    (property "Value" "J" (id 1) (at 207.01 135.89 0)
+      (effects (font (size 1.27 1.27)) hide)
+    )
+    (property "Footprint" "Jumper:SolderJumper-2_P1.3mm_Open_RoundedPad1.0x1.5mm" (id 2) (at 203.2 137.16 0)
+      (effects (font (size 1.27 1.27)) hide)
+    )
+    (property "Datasheet" "~" (id 3) (at 203.2 137.16 0)
+      (effects (font (size 1.27 1.27)) hide)
+    )
+    (pin "1")
+    (pin "2")
+  )
   (symbol (lib_id "power:GND") (at 147.32 87.63 180) (unit 1)
     (in_bom yes) (on_board yes) (fields_autoplaced)
@@
     (pin "2")
   )
+  (symbol (lib_id "Jumper:SolderJumper_2_Open") (at 203.2 140.97 0) (unit 1)
+    (in_bom yes) (on_board yes)
+    (property "Reference" "JP12" (id 0) (at 199.39 139.7 0))
+    (property "Value" "J" (id 1) (at 207.01 139.7 0)
+      (effects (font (size 1.27 1.27)) hide)
+    )
+    (property "Footprint" "Jumper:SolderJumper-2_P1.3mm_Open_RoundedPad1.0x1.5mm" (id 2) (at 203.2 140.97 0)
+      (effects (font (size 1.27 1.27)) hide)
+    )
+    (property "Datasheet" "~" (id 3) (at 203.2 140.97 0)
+      (effects (font (size 1.27 1.27)) hide)
+    )
+    (pin "1")
+    (pin "2")
+  )
   (symbol (lib_id "Device:R") (at 69.85 241.3 270) (mirror x) (unit 1)
     (in_bom yes) (on_board yes)
@@
       (reference "JP9") (unit 1) (value "SolderJumper_3_Open") (footprint "LIBS:SolderJumper-3_P1.3mm_Open_RoundedPad1.0x1.5mm")
     )
+    (path "/580639aa-8bf0-4bdb-a1c6-b4e898ce8bd3"
+      (reference "JP10") (unit 1) (value "J") (footprint "Jumper:SolderJumper-2_P1.3mm_Open_RoundedPad1.0x1.5mm")
+    )
+    (path "/4da549da-bcc2-49a5-ad9e-4ab15d9ce4fe"
+      (reference "JP11") (unit 1) (value "J") (footprint "Jumper:SolderJumper-2_P1.3mm_Open_RoundedPad1.0x1.5mm")
+    )
+    (path "/8e02e558-d089-4537-8518-f8c2b10b979b"
+      (reference "JP12") (unit 1) (value "J") (footprint "Jumper:SolderJumper-2_P1.3mm_Open_RoundedPad1.0x1.5mm")
+    )
+    (path "/406303ee-f65c-4bce-8158-376d04fdc818"
+      (reference "JP13") (unit 1) (value "J") (footprint "Jumper:SolderJumper-2_P1.3mm_Open_RoundedPad1.0x1.5mm")
+    )
     (path "/af94605c-a040-4d97-ba38-cf0c6aa53ef8"

Commit message: .
Parts:
- added J21: Conn_01x01_Female, Connector_Pin:Pin_D0.7mm_L6.5mm_W1.8mm_FlatFork, symbol Connector:Conn_01x01_Female
- added R45: 300, Resistor_SMD:R_0805_2012Metric_Pad1.20x1.40mm_HandSolder, symbol Device:R
Connections:
- net at D6.2 (A), R43.1: now also R45.1
- new net: J21.1 (Pin_1), R45.2
Changed lines of the file:
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@@
   (junction (at 222.25 182.88) (diameter 0) (color 0 0 0 0)
   )
+  (junction (at 250.19 264.16) (diameter 0) (color 0 0 0 0)
+  )
   (junction (at 243.84 142.24) (diameter 0) (color 0 0 0 0)
   )
@@
     (stroke (width 0) (type default) (color 0 0 0 0))
   )
+  (wire (pts (xy 257.81 252.73) (xy 257.81 254))
+    (stroke (width 0) (type default) (color 0 0 0 0))
+  )
   (wire (pts (xy 151.13 20.32) (xy 163.83 20.32))
     (stroke (width 0) (type default) (color 0 0 0 0))
@@
     (stroke (width 0) (type default) (color 0 0 0 0))
   )
+  (wire (pts (xy 250.19 264.16) (xy 257.81 264.16))
+    (stroke (width 0) (type default) (color 0 0 0 0))
+  )
   (wire (pts (xy 110.49 55.88) (xy 123.19 55.88))
     (stroke (width 0) (type default) (color 0 0 0 0))
@@
     (stroke (width 0) (type default) (color 0 0 0 0))
   )
+  (wire (pts (xy 257.81 264.16) (xy 257.81 261.62))
+    (stroke (width 0) (type default) (color 0 0 0 0))
+  )
   (wire (pts (xy 30.48 165.1) (xy 46.99 165.1))
     (stroke (width 0) (type default) (color 0 0 0 0))
@@
     (stroke (width 0) (type default) (color 0 0 0 0))
   )
+  (wire (pts (xy 260.35 252.73) (xy 257.81 252.73))
+    (stroke (width 0) (type default) (color 0 0 0 0))
+  )
   (wire (pts (xy 107.95 119.38) (xy 107.95 121.92))
     (stroke (width 0) (type default) (color 0 0 0 0))
@@
     (pin "2")
   )
+  (symbol (lib_id "Connector:Conn_01x01_Female") (at 265.43 252.73 0) (unit 1)
+    (in_bom yes) (on_board yes) (fields_autoplaced)
+    (property "Reference" "J21" (id 0) (at 266.1412 253.1638 0)
+      (effects (font (size 1.27 1.27)) (justify left))
+    )
+    (property "Value" "Conn_01x01_Female" (id 1) (at 266.1412 254.4322 0)
+      (effects (font (size 1.27 1.27)) (justify left) hide)
+    )
+    (property "Footprint" "Connector_Pin:Pin_D0.7mm_L6.5mm_W1.8mm_FlatFork" (id 2) (at 265.43 252.73 0)
+      (effects (font (size 1.27 1.27)) hide)
+    )
+    (property "Datasheet" "~" (id 3) (at 265.43 252.73 0)
+      (effects (font (size 1.27 1.27)) hide)
+    )
+    (pin "1")
+  )
   (symbol (lib_id "Device:R") (at 68.58 62.23 90) (unit 1)
     (in_bom yes) (on_board yes)
@@
     (pin "1")
   )
+  (symbol (lib_id "Device:R") (at 257.81 257.81 180) (unit 1)
+    (in_bom yes) (on_board yes)
+    (property "Reference" "R45" (id 0) (at 261.62 256.54 0))
+    (property "Value" "300" (id 1) (at 257.81 257.81 90))
+    (property "Footprint" "Resistor_SMD:R_0805_2012Metric_Pad1.20x1.40mm_HandSolder" (id 2) (at 259.588 257.81 90)
+      (effects (font (size 1.27 1.27)) hide)
+    )
+    (property "Datasheet" "~" (id 3) (at 257.81 257.81 0)
+      (effects (font (size 1.27 1.27)) hide)
+    )
+    (pin "1")
+    (pin "2")
+  )
   (symbol (lib_id "Device:R") (at 78.74 82.55 90) (unit 1)
     (in_bom yes) (on_board yes)
@@
       (reference "J20") (unit 1) (value "Conn_01x02") (footprint "Connector_PinHeader_2.54mm:PinHeader_1x02_P2.54mm_Vertical")
     )
+    (path "/56c5990e-0a8e-4c21-9364-f816232ce6ce"
+      (reference "J21") (unit 1) (value "Conn_01x01_Female") (footprint "Connector_Pin:Pin_D0.7mm_L6.5mm_W1.8mm_FlatFork")
+    )
     (path "/7813d41d-0fb2-4ae2-9cd2-80bee7140c73"
       (reference "JP1") (unit 1) (value "R_J") (footprint "Jumper:SolderJumper-2_P1.3mm_Open_RoundedPad1.0x1.5mm")
@@
       (reference "R44") (unit 1) (value "10k") (footprint "Resistor_SMD:R_0805_2012Metric_Pad1.20x1.40mm_HandSolder")
     )
+    (path "/5b04755f-8f83-45b4-a8e3-1c04d011efbd"
+      (reference "R45") (unit 1) (value "300") (footprint "Resistor_SMD:R_0805_2012Metric_Pad1.20x1.40mm_HandSolder")
+    )
     (path "/46d595f4-edb0-4ded-805c-1668608db359"

Commit message: usb comb
Other:
- moved on the sheet: JP6, JP7, JP8, JP9
