File: 19RPI24/19RPI24.kicad_pcb (KiCad board)
At the start: 2 copper layers, 56 x 85 mm, 132 parts, among them CN1 locked, J1 VGA, J10 AudioJack4, J11 USB_B_Micro, J12 Mini-DIN-6, J13 Mini-DIN-6, J14 Conn_01x07, J15 Conn_01x01_Female, J16 USB, J17 Conn_01x02_Female, J18 Conn_01x02_Female, J19 Conn_01x02, J2 EXT, J20 Conn_01x02, J21 Conn_01x01_Female, J3 A_OUT, J4 UART, J5 Micro_SD_Card, J6 Conn_SD, J7 Conn_01x01, J8 USB_A_Stacked, J9 USB_A_Stacked, Q1 BC850, Q2 BC850, Q3 BC850, Q4 BC850, U1 raspberrypi-pico-module, U2 FE1.1s, U3 MW7211A, U4 PSRAM, U5 TDA1387T, U6 LM1117-3.3, Y1 12MHz, Y2 12MHz

Commit message: .
Parts:
- C16: footprint Capacitor_SMD:C_0805_2012Metric_Pad1.18x1.45mm_HandSolder -> Capacitor_Tantalum_SMD:CP_EIA-3528-21_Kemet-B_Pad1.50x2.35mm_HandSolder
- moved C16 0.75 mm to (59.0, 59.3), turned to 90 degrees
- moved JP3 0.37 mm to (40.3, 61.5)
- moved JP2 0.37 mm to (40.3, 66.5)
- turned C22 to -90 degrees
Connections:
- C16 pad 1: GND -> /+5VA
- C16 pad 2: /+5VA -> GND
- C22 pad 1: GND -> /+5VA
- C22 pad 2: /+5VA -> GND
Routing:
- net /+5VA: track 34.5 -> 32.5 mm
Other:
- board text added: "3V3_PICO_EN"
- board text removed: "3V3_I_EN"
