File: 19RPI24/19RPI24.kicad_pcb (KiCad board)
At the start: 2 copper layers, 56 x 85 mm, 132 parts, among them CN1 locked, J1 VGA, J10 AudioJack4, J11 USB_B_Micro, J12 Mini-DIN-6, J13 Mini-DIN-6, J14 Conn_01x07, J15 Conn_01x01_Female, J16 USB, J17 Conn_01x02_Female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

Commit message: .
Parts:
- C16: value 10u -> 220u
- R47: value 10 -> 68
- moved G*** 0.11 mm to (59.9, 39.3)
Routing:
- net GND: track 789.7 -> 814.8 mm, vias 64 -> 66
- net Net-(C6-Pad2): track 10.8 -> 12.5 mm
- net /GP_4: track 27.7 -> 26.7 mm
- net /GP_28: track 23.7 -> 23.0 mm
