File: 19RPI24/19RPI24.kicad_sch (KiCad schematic)
At the start: 128 parts, among them CN1 HDMI, J1 VGA, J10 AudioJack4, J11 USB_B_Micro, J12 Mini-DIN-6, J13 Mini-DIN-6, J14 Conn_01x07, J15 Conn_01x01_Female, J16 USB, J17 Conn_01x02_Female, J18 Conn_01x02_Female, J19 Conn_01x02, J2 EXT, J20 Conn_01x02, J21 Conn_01x01_Female, J3 A_OUT, J4 UART, J5 Micro_SD_Card, J6 Conn_SD, J7 Conn_01x01, J8 USB_A_Stacked, J9 USB_A_Stacked, Q1 BC850, Q2 BC850, Q3 BC850, Q4 BC850, U1 raspberrypi-pico-module, U2 FE1.1s, U3 MW7211A, U4 PSRAM, U5 TDA1387T, U6 LM1117-3.3, Y1 12MHz, Y2 12MHz

Commit message: .
Parts:
- C16: footprint Capacitor_SMD:C_0805_2012Metric_Pad1.18x1.45mm_HandSolder -> Capacitor_Tantalum_SMD:CP_EIA-3528-21_Kemet-B_Pad1.50x2.35mm_HandSolder
Connections:
- net +5VA: now also C16.1, C22.1; no longer C16.2, C22.2
- net GND: now also C16.2, C22.2; no longer C16.1, C22.1
Other:
- moved on the sheet: C16, C22
Changed lines of the file:
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@@
     (pin "9")
   )
-  (symbol (lib_id "Device:C") (at 170.18 219.71 180) (unit 1)
-    (in_bom yes) (on_board yes)
-    (property "Reference" "C22" (id 0) (at 173.99 222.25 0)
-      (effects (font (size 1.27 1.27)) (justify left))
-    )
-    (property "Value" "220u" (id 1) (at 175.26 217.17 0)
-      (effects (font (size 1.27 1.27)) (justify left))
-    )
-    (property "Footprint" "Capacitor_Tantalum_SMD:CP_EIA-6032-28_Kemet-C" (id 2) (at 169.2148 215.9 0)
+  (symbol (lib_id "Device:C") (at 170.18 219.71 0) (unit 1)
+    (in_bom yes) (on_board yes)
+    (property "Reference" "C22" (id 0) (at 170.18 222.25 0)
+      (effects (font (size 1.27 1.27)) (justify left))
+    )
+    (property "Value" "220u" (id 1) (at 170.3923 217.1011 0)
+      (effects (font (size 1.27 1.27)) (justify left))
+    )
+    (property "Footprint" "Capacitor_Tantalum_SMD:CP_EIA-6032-28_Kemet-C" (id 2) (at 171.1452 223.52 0)
       (effects (font (size 1.27 1.27)) hide)
     )
@@
     (pin "2")
   )
-  (symbol (lib_id "Device:C") (at 280.67 77.47 270) (unit 1)
-    (in_bom yes) (on_board yes)
-    (property "Reference" "C16" (id 0) (at 281.94 74.93 90)
-      (effects (font (size 1.27 1.27)) (justify left))
-    )
-    (property "Value" "10u" (id 1) (at 275.59 74.93 90)
-      (effects (font (size 1.27 1.27)) (justify left))
-    )
-    (property "Footprint" "Capacitor_SMD:C_0805_2012Metric_Pad1.18x1.45mm_HandSolder" (id 2) (at 276.86 78.4352 0)
+  (symbol (lib_id "Device:C") (at 280.67 77.47 90) (unit 1)
+    (in_bom yes) (on_board yes)
+    (property "Reference" "C16" (id 0) (at 279.4 80.01 90)
+      (effects (font (size 1.27 1.27)) (justify left))
+    )
+    (property "Value" "10u" (id 1) (at 285.75 80.01 90)
+      (effects (font (size 1.27 1.27)) (justify left))
+    )
+    (property "Footprint" "Capacitor_Tantalum_SMD:CP_EIA-3528-21_Kemet-B_Pad1.50x2.35mm_HandSolder" (id 2) (at 284.48 76.5048 0)
       (effects (font (size 1.27 1.27)) hide)
     )
@@
     )
     (path "/ee402a77-771e-43c1-8557-85fa0a44c13a"
-      (reference "C16") (unit 1) (value "10u") (footprint "Capacitor_SMD:C_0805_2012Metric_Pad1.18x1.45mm_HandSolder")
+      (reference "C16") (unit 1) (value "10u") (footprint "Capacitor_Tantalum_SMD:CP_EIA-3528-21_Kemet-B_Pad1.50x2.35mm_HandSolder")
     )
     (path "/9f980a85-2a09-499d-8750-a2f61ef747c6"

Commit message: .
Parts:
- C16: value 10u -> 220u
- R47: value 10 -> 68
Changed lines of the file:
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@@
     (in_bom yes) (on_board yes)
     (property "Reference" "R47" (id 0) (at 269.24 69.85 90))
-    (property "Value" "10" (id 1) (at 269.24 72.39 90))
+    (property "Value" "68" (id 1) (at 269.24 72.39 90))
     (property "Footprint" "Resistor_SMD:R_0805_2012Metric_Pad1.20x1.40mm_HandSolder" (id 2) (at 269.24 70.612 90)
       (effects (font (size 1.27 1.27)) hide)
@@
     (pin "9")
   )
-  (symbol (lib_id "Device:C") (at 170.18 219.71 0) (unit 1)
+  (symbol (lib_name "C_5") (lib_id "Device:C") (at 170.18 219.71 0) (unit 1)
     (in_bom yes) (on_board yes)
     (property "Reference" "C22" (id 0) (at 170.18 222.25 0)
@@
     (pin "2")
   )
-  (symbol (lib_id "Device:C") (at 280.67 77.47 90) (unit 1)
-    (in_bom yes) (on_board yes)
-    (property "Reference" "C16" (id 0) (at 279.4 80.01 90)
-      (effects (font (size 1.27 1.27)) (justify left))
-    )
-    (property "Value" "10u" (id 1) (at 285.75 80.01 90)
-      (effects (font (size 1.27 1.27)) (justify left))
-    )
-    (property "Footprint" "Capacitor_Tantalum_SMD:CP_EIA-3528-21_Kemet-B_Pad1.50x2.35mm_HandSolder" (id 2) (at 284.48 76.5048 0)
+  (symbol (lib_name "C_4") (lib_id "Device:C") (at 280.67 77.47 90) (mirror x) (unit 1)
+    (in_bom yes) (on_board yes)
+    (property "Reference" "C16" (id 0) (at 285.75 76.2 90)
+      (effects (font (size 1.27 1.27)) (justify left))
+    )
+    (property "Value" "220u" (id 1) (at 279.4 76.2 90)
+      (effects (font (size 1.27 1.27)) (justify left))
+    )
+    (property "Footprint" "Capacitor_Tantalum_SMD:CP_EIA-3528-21_Kemet-B_Pad1.50x2.35mm_HandSolder" (id 2) (at 279.7048 81.28 0)
       (effects (font (size 1.27 1.27)) hide)
     )
@@
     )
     (path "/ee402a77-771e-43c1-8557-85fa0a44c13a"
-      (reference "C16") (unit 1) (value "10u") (footprint "Capacitor_Tantalum_SMD:CP_EIA-3528-21_Kemet-B_Pad1.50x2.35mm_HandSolder")
+      (reference "C16") (unit 1) (value "220u") (footprint "Capacitor_Tantalum_SMD:CP_EIA-3528-21_Kemet-B_Pad1.50x2.35mm_HandSolder")
     )
     (path "/9f980a85-2a09-499d-8750-a2f61ef747c6"
@@
     )
     (path "/1d8ea862-622e-4838-9658-7c6a155ebbb1"
-      (reference "R47") (unit 1) (value "10") (footprint "Resistor_SMD:R_0805_2012Metric_Pad1.20x1.40mm_HandSolder")
+      (reference "R47") (unit 1) (value "68") (footprint "Resistor_SMD:R_0805_2012Metric_Pad1.20x1.40mm_HandSolder")
     )
     (path "/46d595f4-edb0-4ded-805c-1668608db359"
